Commit message: Updated config and bringup to connect moveit with isaac

File: so-arm/so101_ws/src/so101_moveit_config/config/so101_new_calib.ros2_control copy.xacro (robot description, xacro)
@@ -1,25 +1,19 @@
 <?xml version="1.0"?>
 <robot xmlns:xacro="http://www.ros.org/wiki/xacro">
-    <!-- Added 'use_isaac' param alongside existing use_fake_hardware.
-         Call with use_isaac:=true  → TopicBasedSystem bridging /isaac_joint_states + /isaac_joint_command
-            use_fake_hardware:=true → mock_components/GenericSystem (standalone testing)
-            both false             → real SO-ARM serial hardware
-    -->
-    <xacro:macro name="so101_new_calib_ros2_control" params="name initial_positions_file use_fake_hardware use_isaac:=false">
+    <xacro:macro name="so101_new_calib_ros2_control" params="name initial_positions_file use_fake_hardware">
         <xacro:property name="initial_positions" value="${xacro.load_yaml(initial_positions_file)['initial_positions']}"/>
         <ros2_control name="${name}" type="system">
             <hardware>
-                <!-- Isaac Sim mode -->
-                <xacro:if value="${use_isaac}">
+                <xacro:if value="${use_fake_hardware}">
+                    <!-- <plugin>mock_components/GenericSystem</plugin> -->
                     <plugin>topic_based_ros2_control/TopicBasedSystem</plugin>
                     <param name="joint_states_topic">/isaac_joint_states</param>
                     <param name="joint_commands_topic">/isaac_joint_command</param>
+                    <!-- <plugin>topic_based_ros2_control/TopicBasedSystem</plugin> -->
+                    <!-- <param name="joint_states_topic">/isaac_joint_states</param>
+                    <param name="joint_commands_topic">/isaac_joint_command</param>
+                    <param name="sum_wrapped_joint_states">true</param> -->
                 </xacro:if>
-                <!-- Fake/mock hardware (standalone testing without Isaac) -->
-                <xacro:if value="${use_fake_hardware and not use_isaac}">
-                    <plugin>mock_components/GenericSystem</plugin>
-                </xacro:if>
-                <!-- Real SO-ARM serial hardware -->
-                <xacro:unless value="${use_fake_hardware or use_isaac}">
+                <xacro:unless value="${use_fake_hardware}">
                     <plugin>so_arm_100_controller/SOARM100Interface</plugin>
                     <param name="use_serial">true</param>

File: so-arm/so101_ws/src/so101_moveit_config/config/so101_new_calib.urdf.xacro (robot description, xacro)
@@ -3,8 +3,9 @@
     <xacro:arg name="initial_positions_file" default="initial_positions.yaml" />
     <xacro:arg name="use_fake_hardware" default="true" />
+    <xacro:arg name="use_isaac" default="false" />
     <!-- Import so101_new_calib urdf file -->
     <xacro:include filename="$(find so101_description)/urdf/so101_new_calib.urdf" />
     <!-- Import control_xacro -->
     <xacro:include filename="so101_new_calib.ros2_control.xacro" />
-    <xacro:so101_new_calib_ros2_control name="FakeSystem" initial_positions_file="$(arg initial_positions_file)" use_fake_hardware="$(arg use_fake_hardware)"/>
+    <xacro:so101_new_calib_ros2_control name="FakeSystem" initial_positions_file="$(arg initial_positions_file)" use_fake_hardware="$(arg use_fake_hardware)" use_isaac="$(arg use_isaac)"/>
 </robot>
